File: doggedness_schemetic/doggedness_schemetic.kicad_pcb (KiCad board)
At the start: 2 copper layers, 91.2 x 75.9 mm, 35 parts, among them J1 Conn_01x02, J10 TELEMETRY_UART, J11 5V_OUTLET, J2 MOTOR_FL, J3 MOTOR_FR, J4 MOTOR_RL, J5 MOTOR_RR, J6 GY-9250, J7 Screw_Terminal_01x02, J8 SPARE_UART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

Commit message: Add copper pour
Routing:
- added copper zone on B.Cu, net GND
- added copper zone on F.Cu, net GND
Changed lines of the file:
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@@
   (segment (start 152.654 121.539) (end 148.399 117.284) (width 0.25) (layer "F.Cu") (net 80))
   (segment (start 148.399 117.284) (end 148.399 104.902) (width 0.25) (layer "F.Cu") (net 80))
+  (zone (net 1) (net_name "GND") (layers "F&B.Cu") (hatch edge 0.5)
+    (connect_pads thru_hole_only (clearance 0.5))
+    (min_thickness 0.25) (filled_areas_thickness no)
+    (fill yes (thermal_gap 0.5) (thermal_bridge_width 0.5))
+    (polygon
+      (pts
+        (xy 118.872 125.603)
+        (xy 208.915 125.476)
+        (xy 208.915 50.927)
+        (xy 118.872 50.927)
+      )
+    )
+  )
 )
