File: doggedness_schemetic/doggedness_schemetic.kicad_sch (KiCad schematic)
At the start: 35 parts, among them J1 Conn_01x02, J11 5V_OUTLET, J2 GY-9250, J2 MOTOR_FL, J3 CONSOLE_UART, J3 MOTOR_FR, J3 TELEMETRY_UART, J4 MOTOR_RL, J5 MOTOR_RR, J7 Screw_Terminal_01x02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

Commit message: Add README
Other:
- title: (none) -> Doggedness (Chiljeonpalgi) ECU board
Changed lines of the file:
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@@
 (kicad_sch (version 20230121) (generator eeschema)
   (paper "A4")
+  (title_block
+    (title "Doggedness (Chiljeonpalgi) ECU board")
+    (rev "1")
+  )
   (junction (at 60.96 177.8) (diameter 0) (color 0 0 0 0)
   )
